Commit message: balloon remodeling

File: mbzirc_gazebo/models/unit_sphere_0/balloon.urdf (robot description, URDF)
Before this commit: robot my_robot, 2 links, 1 joints
Joints:
- joint balloon_joint: limit lower=-2 upper=10 effort=10 velocity=5 -> lower=0 upper=10 effort=10 velocity=5; origin xyz=0 0 2.0 rpy=0 -1.57 0 -> xyz=0 0 2.0 rpy=0 0 3.1416; type prismatic -> floating
